File: GSE-IGN.kicad_sch (KiCad schematic)
At the start: 25 parts, among them J1 Conn_01x02, J2 DCDC-Regulator-12Vto3.3V, J3 debug-sw1, J4 RJ45, J5 Igniter-1, J6 debug-sw1, Q1 BSS138, U1 Pico, U3 TLP241A

Commit message: 色々変更
Parts:
- added D7: LED, LED_THT:LED_D3.0mm, symbol Device:LED
- added D8: 1N4007, Diode_THT:D_DO-41_SOD81_P10.16mm_Horizontal, symbol Diode:1N4007
- added J7: Igniter-2, Connector_AMASS:AMASS_XT60-M_1x02_P7.20mm_Vertical, symbol Connector_Generic:Conn_01x02
- added JP1: Jumper_2_Open, Connector_PinSocket_2.54mm:PinSocket_1x02_P2.54mm_Vertical, symbol Jumper:Jumper_2_Open
- added R9: 1k, Resistor_THT:R_Axial_DIN0207_L6.3mm_D2.5mm_P7.62mm_Horizontal, symbol Device:R_Small
- C1, C7: footprint (none) -> Capacitor_SMD:C_0805_2012Metric_Pad1.18x1.45mm_HandSolder
- D1: value 45V2A SBM245L -> 45V10A SBM1045VSS; footprint Diode_THT:D_DO-41_SOD81_P10.16mm_Horizontal -> Diode_THT:D_DO-41_SOD81_P12.70mm_Horizontal
- D2: footprint (none) -> Diode_THT:D_DO-41_SOD81_P10.16mm_Horizontal
- D5, D6: footprint (none) -> LED_THT:LED_D3.0mm
- J4: footprint (none) -> Connector_RJ:RJ45_Wuerth_7499010211A_Horizontal
- J5: footprint Connector_JST:JST_XH_B2B-XH-A_1x02_P2.50mm_Vertical -> Connector_AMASS:AMASS_XT60-M_1x02_P7.20mm_Vertical
- R1, R2, R3, R4, R5, R6, R7, R8: footprint (none) -> Resistor_THT:R_Axial_DIN0207_L6.3mm_D2.5mm_P7.62mm_Horizontal
- U1: footprint MCU_RaspberryPi_and_Boards:RPi_Pico_SMD_TH -> KiCad-RP-Pico-main:RPi_Pico_SMD_TH
- U3: value TLP241A -> TLP3543A; footprint Package_DIP:DIP-4_W7.62mm_LongPads -> Package_DIP:DIP-6_W7.62mm; symbol Relay_SolidState:TLP222A -> my_symbol:TLP3543ATP1_F
Connections:
- net +12V: now also U3.6; no longer U3.4
- net +3.3V: now also JP1.2 (B)
- net GND: now also D7.1 (K), D8.2 (A), J7.1 (Pin_1)
- net Igniter-signal: now also JP1.1 (A)
- net at D3.1 (K), J5.2 (Pin_2), R5.2: now also U3.5; no longer U3.3
- net RS232C/RS232C-RX-IN renamed RS485/B
- net RS232C/RS232C-TX-OUT renamed RS485/A
- new net: D8.1 (K), J7.2 (Pin_2), R9.2, U3.4
- new net: D7.2 (A), R9.1
- no-connect marks 0 -> 31
Other:
- removed sheet RS232C
- added sheet RS485 (RS485.kicad_sch)
- moved on the sheet: C7, D2, D3, D5, J4, J5, Q1, R1, R2, R3, R4, R5

Commit message: schはたぶん完成
Parts:
- added C3: 0.1u, Capacitor_SMD:C_0402_1005Metric, symbol Device:C_Small
- added C4: 10u, Capacitor_THT:CP_Radial_D4.0mm_P1.50mm, symbol Device:C_Small
- added J8: RJ45, Connector_RJ:RJ45_Wuerth_7499010211A_Horizontal, symbol Connector:RJ45
- added J9: Conn_01x04_Socket, Connector_PinSocket_1.00mm:PinSocket_1x04_P1.00mm_Vertical, symbol Connector:Conn_01x04_Socket
- C1: value 10u -> 0.1u; footprint Capacitor_SMD:C_0805_2012Metric_Pad1.18x1.45mm_HandSolder -> Diode_SMD:D_0402_1005Metric
- C7: footprint Capacitor_SMD:C_0805_2012Metric_Pad1.18x1.45mm_HandSolder -> Capacitor_THT:CP_Radial_D5.0mm_P2.00mm
- D1: footprint Diode_THT:D_DO-41_SOD81_P12.70mm_Horizontal -> 0000_my_footprint:SBM1060LSS_P20mm_Horizontal
- J2: value DCDC-Regulator-12Vto3.3V -> LD1117S50; footprint Connector_PinSocket_2.54mm:PinSocket_1x03_P2.54mm_Horizontal -> Package_TO_SOT_SMD:SOT-223-3_TabPin2; symbol Connector:Conn_01x03_Socket -> Regulator_Linear:LD1117S50TR_SOT223
- R3: value 240 -> 500
- U1: value Pico -> ATMEGA328P-PU; footprint KiCad-RP-Pico-main:RPi_Pico_SMD_TH -> Package_DIP:DIP-28_W7.62mm; symbol MCU_RaspberryPi_and_Boards:Pico -> MCU_Microchip_ATmega:ATmega328P-P
Connections:
- net +12V: now also D3.1 (K), D8.1 (K), J5.2 (Pin_2), J7.2 (Pin_2), R5.2, R9.2; no longer U3.6
- net Debug-sw1: now also U1.11 (PD5); no longer U1.4 (GPIO2)
- net Debug-sw2: now also U1.12 (PD6); no longer U1.5 (GPIO3)
- net GND: now also J2.1 (GND), U1.22 (GND), U3.5, C3.2, C4.2, J8.1, J8.2, J8.7, J8.8; no longer D3.2 (A), D5.1 (K), D7.1 (K), D8.2 (A), J2.2 (Pin_2), J4.4, J4.5, J5.1 (Pin_1), J7.1 (Pin_1), U1.13 (GND), U1.18 (GND), U1.23 (GND), U1.28 (GND), U1.3 (GND), U1.38 (GND), U1.42 (GND)
- net Igniter-signal: now also U1.6 (PD4); no longer U1.14 (GPIO10)
- net RS232C-TX-IN: now also U1.3 (PD1); no longer U1.1 (GPIO0)
- net RS485/A: now also J4.5, J8.5; no longer J4.6
- net RS485/B: now also J4.4, J8.4; no longer J4.3
- net at D4.1 (K): now also U1.20 (AVCC), U1.7 (VCC), C3.1; no longer U1.39 (VSYS)
- net at U1.15 (PB1): now also J9.1 (Pin_1)
- net at U1.16 (PB2): now also J9.2 (Pin_2)
- net at U1.17 (PB3): now also J9.3 (Pin_3)
- net +3.3V renamed +5V
- net +5V: now also J2.2 (VO), C4.1; no longer J2.1 (Pin_1)
- new net: D7.1 (K), D8.2 (A), J7.1 (Pin_1), U3.4
- new net: D3.2 (A), D5.1 (K), J5.1 (Pin_1), U3.6
- new net: J9.4 (Pin_4), U1.1 (~{RESET}/PC6)
- new net RS485_*RE: U1.5 (PD3)
- new net RS485_DE: U1.4 (PD2)
- no-connect marks 31 -> 17
Other:
- moved on the sheet: C1, C7, D1, D3, D4, D5, D6, D7, D8, J1, J5, J7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

Commit message: アートワーク終わり
Parts:
- added C5, C6: 22p, Capacitor_SMD:C_0603_1608Metric, symbol Device:C_Small
- added Y1: Crystal_GND3_Small, Crystal:Crystal_HC49-4H_Vertical, symbol Device:Crystal_Small
- C1: value 0.1u -> 10u; footprint Diode_SMD:D_0402_1005Metric -> Capacitor_THT:CP_Radial_D4.0mm_P1.50mm
- J4, J8: footprint Connector_RJ:RJ45_Wuerth_7499010211A_Horizontal -> 0000_my_footprint:78108P8C
- J9: footprint Connector_PinSocket_1.00mm:PinSocket_1x04_P1.00mm_Vertical -> Connector_PinSocket_2.54mm:PinSocket_1x04_P2.54mm_Vertical
- JP1: footprint Connector_PinSocket_2.54mm:PinSocket_1x02_P2.54mm_Vertical -> Connector_JST:JST_XH_B2B-XH-A_1x02_P2.50mm_Vertical
Connections:
- net +5V: now also JP1.1 (A); no longer JP1.2 (B)
- net GND: now also C5.2, C6.2
- net Igniter-signal: now also JP1.2 (B); no longer JP1.1 (A)
- net RS485/A: now also J4.6, J8.6; no longer J4.5, J8.5
- net at U1.10 (XTAL2/PB7): now also C6.1, Y1.1
- net at U1.9 (XTAL1/PB6): now also C5.1, Y1.2
- no-connect marks 17 -> 15
Other:
- moved on the sheet: C1, C4, D1, D2, D6, J1, J2, J4, J8, JP1, Q1, R1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

Commit message: 少し小型化
Parts:
- added R13: 1M, Resistor_THT:R_Axial_DIN0207_L6.3mm_D2.5mm_P7.62mm_Horizontal, symbol Device:R_Small
- C1, C4: value 10u -> 47u
- C3: footprint Capacitor_SMD:C_0402_1005Metric -> Capacitor_SMD:C_0603_1608Metric_Pad1.08x0.95mm_HandSolder
Connections:
- net at C5.1, U1.9 (XTAL1/PB6), Y1.2: now also R13.2
- net at C6.1, U1.10 (XTAL2/PB7), Y1.1: now also R13.1
Other:
- moved on the sheet: C5, C6, Y1
